File: meme-o-clock-pcb.kicad_pcb (KiCad board)
At the start: 4 copper layers, 88 x 100 mm, 24 parts, among them J1 USB_C_Receptacle_USB2.0_16P, J2 Conn_01x04_Pin, J3 Conn_01x02_Pin, J4 Conn_01x03_Pin, SW1 SW_Push, SW2 SW_Push, SW3 SW_Push, SW4 SW_Push, U1 MAX98357A, U2 APDS-9306

Commit message: Autosave
Routing:
- net GND: track 436.3 -> 437.3 mm
Changed lines of the file:
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@@
+	)
+	(segment
+		(start 136.427 92.8)
+		(end 136.427 86.227)
+		(width 0.4)
+		(layer "F.Cu")
+		(net "GND")
 	)
 	(segment
@@
 	(segment
 		(start 136.427 136.0055)
-		(end 136.427 86.227)
+		(end 136.427 92.8)
 		(width 0.4)
 		(layer "F.Cu")
@@
 	)
 	(segment
+		(start 136.644 93.017)
+		(end 137.3625 93.017)
+		(width 0.4)
+		(layer "F.Cu")
+		(net "GND")
+	)
+	(segment
 		(start 122.3 65.25)
 		(end 120.8 63.75)
@@
 		(width 0.4)
 		(layer "F.Cu")
+		(net "GND")
+	)
+	(segment
+		(start 136.427 92.8)
+		(end 136.644 93.017)
+		(width 0.4)
+		(layer "F.Cu")

Commit message: Autosave
Routing:
- net +3V3: track 0.25 -> 81.6 mm, vias 0 -> 1
Changed lines of the file:
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@@
+	)
+	(segment
+		(start 79.611712 99.3)
+		(end 79.155856 99.755856)
+		(width 0.4)
+		(layer "F.Cu")
+		(net "+3V3")
+	)
+	(segment
+		(start 80.8 99.4)
+		(end 80.7 99.3)
+		(width 0.4)
+		(layer "F.Cu")
+		(net "+3V3")
+	)
+	(segment
+		(start 80.875 99.4)
+		(end 80.8 99.4)
+		(width 0.4)
+		(layer "F.Cu")
+		(net "+3V3")
+	)
+	(segment
+		(start 80.7 99.3)
+		(end 79.611712 99.3)
+		(width 0.4)
+		(layer "F.Cu")
+		(net "+3V3")
+	)
+	(via
+		(at 79.155856 99.755856)
+		(size 0.6)
+		(drill 0.3)
+		(layers "F.Cu" "B.Cu")
+		(net "+3V3")
+	)
+	(segment
+		(start 104.355856 99.755856)
+		(end 107.127 102.527)
+		(width 0.4)
+		(layer "B.Cu")
+		(net "+3V3")
+	)
+	(segment
+		(start 79.155856 99.755856)
+		(end 104.355856 99.755856)
+		(width 0.4)
+		(layer "B.Cu")
+		(net "+3V3")
+	)
+	(segment
+		(start 120.2 99.8)
+		(end 120.2 93.1)
+		(width 0.4)
+		(layer "B.Cu")
+		(net "+3V3")
+	)
+	(segment
+		(start 120.2 93.1)
+		(end 118.393 94.907)
+		(width 0.4)
+		(layer "B.Cu")
+		(net "+3V3")
+	)
+	(segment
+		(start 118.393 94.907)
+		(end 106.693 94.907)
+		(width 0.4)
+		(layer "B.Cu")
+		(net "+3V3")
+	)
+	(segment
+		(start 106.693 94.907)
+		(end 96 105.6)
+		(width 0.4)
+		(layer "B.Cu")
+		(net "+3V3")
+	)
+	(segment
+		(start 107.127 102.527)
+		(end 117.473 102.527)
+		(width 0.4)
+		(layer "B.Cu")
+		(net "+3V3")
+	)
+	(segment
+		(start 117.473 102.527)
+		(end 120.2 99.8)
+		(width 0.4)
+		(layer "B.Cu")
+		(net "+3V3")
 	)
 	(segment

Commit message: Autosave
Routing:
- net +3V3: track 81.6 -> 134.6 mm
Changed lines of the file:
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@@
+	)
+	(segment
+		(start 79.6 99.755856)
+		(end 104.355856 99.755856)
+		(width 0.4)
+		(layer "B.Cu")
+		(net "+3V3")
+	)
+	(segment
+		(start 127.613 107.893)
+		(end 128.74 109.02)
+		(width 0.4)
+		(layer "B.Cu")
+		(net "+3V3")
 	)
 	(segment
@@
 	(segment
 		(start 79.155856 99.755856)
-		(end 104.355856 99.755856)
+		(end 79.6 99.755856)
 		(width 0.4)
 		(layer "B.Cu")
@@
 		(start 120.2 99.8)
 		(end 120.2 93.1)
+		(width 0.4)
+		(layer "B.Cu")
+		(net "+3V3")
+	)
+	(segment
+		(start 79.6 99.755856)
+		(end 81.532518 99.755856)
+		(width 0.4)
+		(layer "B.Cu")
+		(net "+3V3")
+	)
+	(segment
+		(start 89.669662 107.893)
+		(end 127.613 107.893)
 		(width 0.4)
 		(layer "B.Cu")
@@
 		(width 0.4)
 		(layer "B.Cu")
+		(net "+3V3")
+	)
+	(segment
+		(start 81.532518 99.755856)
+		(end 89.669662 107.893)
+		(width 0.4)
+		(layer "B.Cu")

Commit message: Autosave
Routing:
- net +3V3: track 134.6 -> 113.6 mm
Changed lines of the file:
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@@
-	)
-	(segment
-		(start 120.2 99.8)
-		(end 120.2 93.1)
-		(width 0.4)
-		(layer "B.Cu")
-		(net "+3V3")
 	)
 	(segment
@@
 		(width 0.4)
 		(layer "B.Cu")
-		(net "+3V3")
-	)
-	(segment
-		(start 120.2 93.1)
-		(end 118.393 94.907)
-		(width 0.4)
-		(layer "B.Cu")
-		(net "+3V3")
-	)
-	(segment
-		(start 118.393 94.907)
-		(end 106.693 94.907)
-		(width 0.4)
-		(layer "B.Cu")

Commit message: Autosave
Routing:
- net +3V3: track 113.6 -> 95.5 mm
Changed lines of the file:
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@@
-	)
-	(segment
-		(start 104.355856 99.755856)
-		(end 107.127 102.527)
-		(width 0.4)
-		(layer "B.Cu")
-		(net "+3V3")
 	)
 	(segment
@@
 		(width 0.4)
 		(layer "B.Cu")
-		(net "+3V3")
-	)
-	(segment
-		(start 107.127 102.527)
-		(end 117.473 102.527)
-		(width 0.4)
-		(layer "B.Cu")
-		(net "+3V3")
-	)
-	(segment
-		(start 117.473 102.527)
-		(end 120.2 99.8)
-		(width 0.4)
-		(layer "B.Cu")

Commit message: Autosave
Routing:
- net +3V3: track 95.5 -> 80.4 mm
Changed lines of the file:
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@@
-	)
-	(segment
-		(start 106.693 94.907)
-		(end 96 105.6)
-		(width 0.4)
-		(layer "B.Cu")
-		(net "+3V3")
 	)
 	(segment

Commit message: Autosave
Routing:
- net +3V3: track 80.4 -> 53.2 mm
Changed lines of the file:
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@@
-	)
-	(segment
-		(start 79.6 99.755856)
-		(end 104.355856 99.755856)
-		(width 0.4)
-		(layer "B.Cu")
-		(net "+3V3")
 	)
 	(segment
@@
 		(width 0.4)
 		(layer "B.Cu")
-		(net "+3V3")
-	)
-	(segment
-		(start 79.155856 99.755856)
-		(end 79.6 99.755856)
-		(width 0.4)
-		(layer "B.Cu")
-		(net "+3V3")
-	)
-	(segment
-		(start 79.6 99.755856)
-		(end 81.532518 99.755856)
-		(width 0.4)
-		(layer "B.Cu")

Commit message: Autosave
Routing:
- net +3V3: track 53.2 -> 0.25 mm, vias 1 -> 0
Changed lines of the file:
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@@
-	)
-	(segment
-		(start 79.611712 99.3)
-		(end 79.155856 99.755856)
-		(width 0.4)
-		(layer "F.Cu")
-		(net "+3V3")
-	)
-	(segment
-		(start 80.8 99.4)
-		(end 80.7 99.3)
-		(width 0.4)
-		(layer "F.Cu")
-		(net "+3V3")
-	)
-	(segment
-		(start 80.875 99.4)
-		(end 80.8 99.4)
-		(width 0.4)
-		(layer "F.Cu")
-		(net "+3V3")
-	)
-	(segment
-		(start 80.7 99.3)
-		(end 79.611712 99.3)
-		(width 0.4)
-		(layer "F.Cu")
-		(net "+3V3")
-	)
-	(via
-		(at 79.155856 99.755856)
-		(size 0.6)
-		(drill 0.3)
-		(layers "F.Cu" "B.Cu")
-		(net "+3V3")
-	)
-	(segment
-		(start 127.613 107.893)
-		(end 128.74 109.02)
-		(width 0.4)
-		(layer "B.Cu")
-		(net "+3V3")
-	)
-	(segment
-		(start 89.669662 107.893)
-		(end 127.613 107.893)
-		(width 0.4)
-		(layer "B.Cu")
-		(net "+3V3")
-	)
-	(segment
-		(start 81.532518 99.755856)
-		(end 89.669662 107.893)
-		(width 0.4)
-		(layer "B.Cu")
-		(net "+3V3")
 	)
 	(segment
