File: meme-o-clock-pcb.kicad_pcb (KiCad board)
At the start: 4 copper layers, 88 x 100 mm, 24 parts, among them J1 USB_C_Receptacle_USB2.0_16P, J2 Conn_01x04_Pin, J3 Conn_01x02_Pin, J4 Conn_01x03_Pin, SW1 SW_Push, SW2 SW_Push, SW3 SW_Push, SW4 SW_Push, U1 MAX98357A, U2 APDS-9306

Commit message: Autosave
Routing:
- net +3V3: track 264.0 -> 316.3 mm, vias 5 -> 6
Changed lines of the file:
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@@
+	)
+	(segment
+		(start 80.875 99.4)
+		(end 80.875 100.197662)
+		(width 0.4)
+		(layer "F.Cu")
+		(net "+3V3")
+	)
+	(segment
+		(start 80.875 100.197662)
+		(end 81.592487 100.915149)
+		(width 0.4)
+		(layer "F.Cu")
+		(net "+3V3")
 	)
 	(segment
@@
 	)
 	(segment
+		(start 81.592487 100.915149)
+		(end 82.73956 100.915149)
+		(width 0.4)
+		(layer "F.Cu")
+		(net "+3V3")
+	)
+	(segment
 		(start 80.875 99.4)
 		(end 80.4 99.4)
@@
 	)
 	(via
+		(at 82.73956 100.915149)
+		(size 0.6)
+		(drill 0.3)
+		(layers "F.Cu" "B.Cu")
+		(net "+3V3")
+	)
+	(via
 		(at 137.405656 91.283)
 		(size 0.6)
@@
 	)
 	(segment
+		(start 82.73956 100.915149)
+		(end 84.637411 102.813)
+		(width 0.4)
+		(layer "B.Cu")
+		(net "+3V3")
+	)
+	(segment
 		(start 133 117.5)
 		(end 133 113.28)
@@
 	)
 	(segment
+		(start 84.637411 102.813)
+		(end 122.533 102.813)
+		(width 0.4)
+		(layer "B.Cu")
+		(net "+3V3")
+	)
+	(segment
 		(start 128.74 109.02)
 		(end 137.405656 100.354344)
@@
 		(width 0.4)
 		(layer "B.Cu")
+		(net "+3V3")
+	)
+	(segment
+		(start 122.533 102.813)
+		(end 128.74 109.02)
+		(width 0.4)
+		(layer "B.Cu")

Commit message: Autosave
Routing:
- net +3V3: track 316.3 -> 264.0 mm, vias 6 -> 5
Changed lines of the file:
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@@
-	)
-	(segment
-		(start 80.875 99.4)
-		(end 80.875 100.197662)
-		(width 0.4)
-		(layer "F.Cu")
-		(net "+3V3")
-	)
-	(segment
-		(start 80.875 100.197662)
-		(end 81.592487 100.915149)
-		(width 0.4)
-		(layer "F.Cu")
-		(net "+3V3")
 	)
 	(segment
@@
 	)
 	(segment
-		(start 81.592487 100.915149)
-		(end 82.73956 100.915149)
-		(width 0.4)
-		(layer "F.Cu")
-		(net "+3V3")
-	)
-	(segment
 		(start 80.875 99.4)
 		(end 80.4 99.4)
@@
 	)
 	(via
-		(at 82.73956 100.915149)
-		(size 0.6)
-		(drill 0.3)
-		(layers "F.Cu" "B.Cu")
-		(net "+3V3")
-	)
-	(via
 		(at 137.405656 91.283)
 		(size 0.6)
@@
 	)
 	(segment
-		(start 82.73956 100.915149)
-		(end 84.637411 102.813)
-		(width 0.4)
-		(layer "B.Cu")
-		(net "+3V3")
-	)
-	(segment
 		(start 133 117.5)
 		(end 133 113.28)
@@
 	)
 	(segment
-		(start 84.637411 102.813)
-		(end 122.533 102.813)
-		(width 0.4)
-		(layer "B.Cu")
-		(net "+3V3")
-	)
-	(segment
 		(start 128.74 109.02)
 		(end 137.405656 100.354344)
@@
 		(width 0.4)
 		(layer "B.Cu")
-		(net "+3V3")
-	)
-	(segment
-		(start 122.533 102.813)
-		(end 128.74 109.02)
-		(width 0.4)
-		(layer "B.Cu")

Commit message: Autosave
Routing:
- net +3V3: track 264.0 -> 268.8 mm, vias 5 -> 6
Changed lines of the file:
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@@
+	)
+	(segment
+		(start 80.1 85.6)
+		(end 79.7 86)
+		(width 0.4)
+		(layer "F.Cu")
+		(net "+3V3")
 	)
 	(segment
@@
 	)
 	(segment
+		(start 80.975 85.6)
+		(end 80.1 85.6)
+		(width 0.4)
+		(layer "F.Cu")
+		(net "+3V3")
+	)
+	(segment
 		(start 80.25 113.65)
 		(end 80.2 113.7)
@@
 	)
 	(via
+		(at 79.7 86)
+		(size 0.6)
+		(drill 0.3)
+		(layers "F.Cu" "B.Cu")
+		(net "+3V3")
+	)
+	(via
 		(at 133 117.5)
 		(size 0.6)
@@
 	)
 	(segment
-		(start 80.6 70)
+		(start 80.6 89)
 		(end 80.6 100.2)
+		(width 0.4)
+		(layer "B.Cu")
+		(net "+3V3")
+	)
+	(segment
+		(start 79.7 88.1)
+		(end 80.6 89)
 		(width 0.4)
 		(layer "B.Cu")
@@
 	)
 	(segment
+		(start 79.7 86)
+		(end 79.7 88.1)
+		(width 0.4)
+		(layer "B.Cu")
+		(net "+3V3")
+	)
+	(segment
 		(start 133 117.5)
 		(end 133 113.28)
@@
 		(width 0.4)
 		(layer "B.Cu")
+		(net "+3V3")
+	)
+	(segment
+		(start 80.6 70)
+		(end 80.6 89)
+		(width 0.4)
+		(layer "B.Cu")

Commit message: Autosave
Routing:
- net +5V: track 16.4 -> 126.9 mm, vias 0 -> 2
Changed lines of the file:
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@@
+	)
+	(segment
+		(start 95.0275 102.0725)
+		(end 94.8 102.3)
+		(width 0.2)
+		(layer "F.Cu")
+		(net "+5V")
+	)
+	(segment
+		(start 95.0275 102.04)
+		(end 95.0275 102.0725)
+		(width 0.2)
+		(layer "F.Cu")
+		(net "+5V")
+	)
+	(segment
+		(start 115.9 137.3)
+		(end 115.9 137.6)
+		(width 0.4)
+		(layer "F.Cu")
+		(net "+5V")
 	)
 	(segment
@@
 	)
 	(segment
+		(start 95.0275 102.04)
+		(end 93.7 103.3675)
+		(width 0.2)
+		(layer "F.Cu")
+		(net "+5V")
+	)
+	(segment
 		(start 96.840001 102.74)
 		(end 97.2525 102.74)
@@
 	)
 	(segment
+		(start 115.9 137.6)
+		(end 116 137.7)
+		(width 0.4)
+		(layer "F.Cu")
+		(net "+5V")
+	)
+	(segment
 		(start 96.202 98.657)
 		(end 96.202 102.1895)
@@
 	)
 	(segment
+		(start 116 136.8)
+		(end 115.3 136.1)
+		(width 0.4)
+		(layer "F.Cu")
+		(net "+5V")
+	)
+	(segment
 		(start 95.7 98.155)
 		(end 96.0275 98.4825)
@@
 		(net "+5V")
 	)
+	(segment
+		(start 116 137.7)
+		(end 116 136.8)
+		(width 0.4)
+		(layer "F.Cu")
+		(net "+5V")
+	)
+	(segment
+		(start 93.7 103.3675)
+		(end 93.7 104.4)
+		(width 0.2)
+		(layer "F.Cu")
+		(net "+5V")
+	)
+	(via
+		(at 93.7 104.4)
+		(size 0.6)
+		(drill 0.3)
+		(layers "F.Cu" "B.Cu")
+		(net "+5V")
+	)
+	(via
+		(at 115.3 136.1)
+		(size 0.6)
+		(drill 0.3)
+		(layers "F.Cu" "B.Cu")
+		(net "+5V")
+	)
+	(segment
+		(start 130.487947 83.62)
+		(end 128.74 83.62)
+		(width 0.2)
+		(layer "B.Cu")
+		(net "+5V")
+	)
+	(segment
+		(start 133.218291 118.027)
+		(end 137.932656 113.312635)
+		(width 0.2)
+		(layer "B.Cu")
+		(net "+5V")
+	)
+	(segment
+		(start 115.3 136.1)
+		(end 115.3 119.027)
+		(width 0.4)
+		(layer "B.Cu")
+		(net "+5V")
+	)
+	(segment
+		(start 107.327 118.027)
+		(end 114.3 118.027)
+		(width 0.2)
+		(layer "B.Cu")
+		(net "+5V")
+	)
+	(segment
+		(start 114.3 118.027)
+		(end 133.218291 118.027)
+		(width 0.2)
+		(layer "B.Cu")
+		(net "+5V")
+	)
+	(segment
+		(start 137.932656 113.312635)
+		(end 137.932656 91.064709)
+		(width 0.2)
+		(layer "B.Cu")
+		(net "+5V")
+	)
+	(segment
+		(start 93.7 104.4)
+		(end 107.327 118.027)
+		(width 0.2)
+		(layer "B.Cu")
+		(net "+5V")
+	)
+	(segment
+		(start 137.932656 91.064709)
+		(end 130.487947 83.62)
+		(width 0.2)
+		(layer "B.Cu")
+		(net "+5V")
+	)
+	(segment
+		(start 115.3 119.027)
+		(end 114.3 118.027)
+		(width 0.4)
+		(layer "B.Cu")
+		(net "+5V")
+	)
