File: meme-o-clock-pcb.kicad_pcb (KiCad board)
At the start: 4 copper layers, 88 x 100 mm, 24 parts, among them J1 USB_C_Receptacle_USB2.0_16P, J2 Conn_01x04_Pin, J3 Conn_01x02_Pin, J4 Conn_01x03_Pin, SW1 SW_Push, SW2 SW_Push, SW3 SW_Push, SW4 SW_Push, U1 MAX98357A, U2 APDS-9306

Commit message: Autosave
Routing:
- net +5V: track 126.9 -> 133.0 mm, vias 2 -> 3
Changed lines of the file:
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@@
+	)
+	(segment
+		(start 125.993592 60.778)
+		(end 126.227 61.011408)
+		(width 0.4)
+		(layer "F.Cu")
+		(net "+5V")
 	)
 	(segment
@@
 		(end 95.0275 102.0725)
 		(width 0.2)
+		(layer "F.Cu")
+		(net "+5V")
+	)
+	(segment
+		(start 121.773 61.011408)
+		(end 122.006408 60.778)
+		(width 0.4)
+		(layer "F.Cu")
+		(net "+5V")
+	)
+	(segment
+		(start 122.006408 60.778)
+		(end 125.993592 60.778)
+		(width 0.4)
+		(layer "F.Cu")
+		(net "+5V")
+	)
+	(segment
+		(start 121.773 61.507)
+		(end 121.773 61.011408)
+		(width 0.4)
 		(layer "F.Cu")
 		(net "+5V")
@@
 	)
 	(segment
+		(start 121.6 61.68)
+		(end 121.773 61.507)
+		(width 0.4)
+		(layer "F.Cu")
+		(net "+5V")
+	)
+	(segment
 		(start 96.202 98.657)
 		(end 96.202 102.1895)
@@
 		(end 96.202 98.657)
 		(width 0.2)
+		(layer "F.Cu")
+		(net "+5V")
+	)
+	(segment
+		(start 126.227 61.507)
+		(end 126.4 61.68)
+		(width 0.4)
 		(layer "F.Cu")
 		(net "+5V")
@@
 		(end 96.0275 98.4825)
 		(width 0.2)
+		(layer "F.Cu")
+		(net "+5V")
+	)
+	(segment
+		(start 126.227 61.011408)
+		(end 126.227 61.507)
+		(width 0.4)
 		(layer "F.Cu")
 		(net "+5V")
@@
 		(size 0.6)
 		(drill 0.3)
+		(layers "F.Cu" "B.Cu")
+		(net "+5V")
+	)
+	(via
+		(at 126.4 61.68)
+		(size 0.6)
+		(drill 0.3)

Commit message: Autosave
Routing:
- net +5V: track 133.0 -> 126.9 mm, vias 3 -> 2
Changed lines of the file:
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@@
-	)
-	(segment
-		(start 125.993592 60.778)
-		(end 126.227 61.011408)
-		(width 0.4)
-		(layer "F.Cu")
-		(net "+5V")
 	)
 	(segment
@@
 		(end 95.0275 102.0725)
 		(width 0.2)
-		(layer "F.Cu")
-		(net "+5V")
-	)
-	(segment
-		(start 121.773 61.011408)
-		(end 122.006408 60.778)
-		(width 0.4)
-		(layer "F.Cu")
-		(net "+5V")
-	)
-	(segment
-		(start 122.006408 60.778)
-		(end 125.993592 60.778)
-		(width 0.4)
-		(layer "F.Cu")
-		(net "+5V")
-	)
-	(segment
-		(start 121.773 61.507)
-		(end 121.773 61.011408)
-		(width 0.4)
 		(layer "F.Cu")
 		(net "+5V")
@@
 	)
 	(segment
-		(start 121.6 61.68)
-		(end 121.773 61.507)
-		(width 0.4)
-		(layer "F.Cu")
-		(net "+5V")
-	)
-	(segment
 		(start 96.202 98.657)
 		(end 96.202 102.1895)
@@
 		(end 96.202 98.657)
 		(width 0.2)
-		(layer "F.Cu")
-		(net "+5V")
-	)
-	(segment
-		(start 126.227 61.507)
-		(end 126.4 61.68)
-		(width 0.4)
 		(layer "F.Cu")
 		(net "+5V")
@@
 		(end 96.0275 98.4825)
 		(width 0.2)
-		(layer "F.Cu")
-		(net "+5V")
-	)
-	(segment
-		(start 126.227 61.011408)
-		(end 126.227 61.507)
-		(width 0.4)
 		(layer "F.Cu")
 		(net "+5V")
@@
 		(size 0.6)
 		(drill 0.3)
-		(layers "F.Cu" "B.Cu")
-		(net "+5V")
-	)
-	(via
-		(at 126.4 61.68)
-		(size 0.6)
-		(drill 0.3)

Commit message: PCB Save
Routing:
- net +5V: track 126.9 -> 162.1 mm, vias 2 -> 3
Changed lines of the file:
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@@
+	)
+	(segment
+		(start 126.4 61.68)
+		(end 126.227 61.507)
+		(width 0.4)
+		(layer "F.Cu")
+		(net "+5V")
 	)
 	(segment
@@
 	)
 	(segment
+		(start 122.984408 59.8)
+		(end 123 59.8)
+		(width 0.4)
+		(layer "F.Cu")
+		(net "+5V")
+	)
+	(segment
 		(start 115.9 137.3)
 		(end 115.9 137.6)
@@
 	)
 	(segment
+		(start 121.773 61.011408)
+		(end 122.984408 59.8)
+		(width 0.4)
+		(layer "F.Cu")
+		(net "+5V")
+	)
+	(segment
 		(start 96.0525 102.04)
 		(end 97.2525 103.24)
@@
 	)
 	(segment
+		(start 125.730592 60.515)
+		(end 122.269408 60.515)
+		(width 0.4)
+		(layer "F.Cu")
+		(net "+5V")
+	)
+	(segment
 		(start 96.0275 101.927499)
 		(end 96.840001 102.74)
@@
 	)
 	(segment
+		(start 121.773 61.011408)
+		(end 121.773 61.507)
+		(width 0.4)
+		(layer "F.Cu")
+		(net "+5V")
+	)
+	(segment
 		(start 95.7 98.155)
 		(end 96.202 98.657)
@@
 	)
 	(segment
+		(start 121.773 61.507)
+		(end 121.6 61.68)
+		(width 0.4)
+		(layer "F.Cu")
+		(net "+5V")
+	)
+	(segment
 		(start 116 136.8)
 		(end 115.3 136.1)
@@
 	)
 	(segment
+		(start 126.227 61.507)
+		(end 126.227 61.011408)
+		(width 0.4)
+		(layer "F.Cu")
+		(net "+5V")
+	)
+	(segment
 		(start 96.202 102.1895)
 		(end 97.2525 103.24)
@@
 	)
 	(segment
+		(start 126.227 61.011408)
+		(end 125.730592 60.515)
+		(width 0.4)
+		(layer "F.Cu")
+		(net "+5V")
+	)
+	(segment
 		(start 116 137.7)
 		(end 116 136.8)
+		(width 0.4)
+		(layer "F.Cu")
+		(net "+5V")
+	)
+	(segment
+		(start 122.269408 60.515)
+		(end 121.773 61.011408)
 		(width 0.4)
 		(layer "F.Cu")
@@
 		(net "+5V")
 	)
+	(via
+		(at 123 59.8)
+		(size 0.6)
+		(drill 0.3)
+		(layers "F.Cu" "B.Cu")
+		(net "+5V")
+	)
 	(segment
 		(start 130.487947 83.62)
@@
 		(layer "B.Cu")
 		(net "+5V")
+	)
+	(segment
+		(start 123 59.8)
+		(end 129.867 66.667)
+		(width 0.4)
+		(layer "B.Cu")
+		(net "+5V")
+	)
+	(segment
+		(start 129.867 82.493)
+		(end 128.74 83.62)
+		(width 0.4)
+		(layer "B.Cu")
+		(net "+5V")
+	)
+	(segment
+		(start 129.867 66.667)
+		(end 129.867 82.493)
+		(width 0.4)
+		(layer "B.Cu")
+		(net "+5V")

Commit message: SCH Save
Routing:
- net Net-(A1-D10/CS): track 0.00 -> 28.8 mm, vias 0 -> 4
- net unconnected-(J1-SHIELD-PadSH): track 0.00 -> 4.39 mm
Changed lines of the file:
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@@
 			(layer "F.Fab")
 		)
-		(fp_text user "${REFERENCE}"
-			(at 0 0 0)
-			(layer "F.Fab")
-			(effects
-				(font
-					(size 0.5 0.5)
-					(thickness 0.08)
-				)
-			)
-		)
 		(pad "1" smd roundrect
 			(at -0.7625 -0.795 180)
@@
 	(footprint "Connector_USB:USB_C_Receptacle_GCT_USB4105-xx-A_16P_TopMnt_Horizontal"
 		(layer "F.Cu")
-		(at 124 58 180)
+		(at 124.01 57.995 180)
 		(descr "USB 2.0 Type C Receptacle, GCT, 16P, top mounted, horizontal, 5A: https://gct.co/files/drawings/usb4105.pdf")
 		(tags "USB C Type-C Receptacle SMD USB 2.0 16P 16C USB4105-15-A USB4105-15-A-060 USB4105-15-A-120 USB4105-GF-A USB4105-GF-A-060 USB4105-GF-A-120")
@@
 	)
 	(segment
+		(start 123.6 103.5)
+		(end 126.8 100.3)
+		(width 0.127)
+		(layer "F.Cu")
+		(net "Net-(A1-D10{slash}CS)")
+	)
+	(segment
+		(start 134.6 93.1)
+		(end 135.235 92.465)
+		(width 0.127)
+		(layer "F.Cu")
+		(net "Net-(A1-D10{slash}CS)")
+	)
+	(segment
+		(start 121.9 103.5)
+		(end 123.6 103.5)
+		(width 0.127)
+		(layer "F.Cu")
+		(net "Net-(A1-D10{slash}CS)")
+	)
+	(segment
+		(start 116.32 106.48)
+		(end 119.4 103.4)
+		(width 0.127)
+		(layer "F.Cu")
+		(net "Net-(A1-D10{slash}CS)")
+	)
+	(segment
+		(start 135.235 92.465)
+		(end 135.8375 92.465)
+		(width 0.127)
+		(layer "F.Cu")
+		(net "Net-(A1-D10{slash}CS)")
+	)
+	(segment
+		(start 113.5 106.48)
+		(end 116.32 106.48)
+		(width 0.127)
+		(layer "F.Cu")
+		(net "Net-(A1-D10{slash}CS)")
+	)
+	(via
+		(at 119.4 103.4)
+		(size 0.6)
+		(drill 0.3)
+		(layers "F.Cu" "B.Cu")
+		(net "Net-(A1-D10{slash}CS)")
+	)
+	(via
+		(at 121.9 103.5)
+		(size 0.6)
+		(drill 0.3)
+		(layers "F.Cu" "B.Cu")
+		(net "Net-(A1-D10{slash}CS)")
+	)
+	(via
+		(at 134.6 93.1)
+		(size 0.6)
+		(drill 0.3)
+		(layers "F.Cu" "B.Cu")
+		(net "Net-(A1-D10{slash}CS)")
+	)
+	(via
+		(at 126.8 100.3)
+		(size 0.6)
+		(drill 0.3)
+		(layers "F.Cu" "B.Cu")
+		(net "Net-(A1-D10{slash}CS)")
+	)
+	(segment
+		(start 126.8 99.399221)
+		(end 128.499221 97.7)
+		(width 0.127)
+		(layer "B.Cu")
+		(net "Net-(A1-D10{slash}CS)")
+	)
+	(segment
+		(start 128.499221 97.7)
+		(end 130 97.7)
+		(width 0.127)
+		(layer "B.Cu")
+		(net "Net-(A1-D10{slash}CS)")
+	)
+	(segment
+		(start 119.4 103.4)
+		(end 121.8 103.4)
+		(width 0.127)
+		(layer "B.Cu")
+		(net "Net-(A1-D10{slash}CS)")
+	)
+	(segment
+		(start 130 97.7)
+		(end 134.6 93.1)
+		(width 0.127)
+		(layer "B.Cu")
+		(net "Net-(A1-D10{slash}CS)")
+	)
+	(segment
+		(start 121.8 103.4)
+		(end 121.9 103.5)
+		(width 0.127)
+		(layer "B.Cu")
+		(net "Net-(A1-D10{slash}CS)")
+	)
+	(segment
+		(start 126.8 100.3)
+		(end 126.8 99.399221)
+		(width 0.127)
+		(layer "B.Cu")
+		(net "Net-(A1-D10{slash}CS)")
+	)
+	(segment
 		(start 95.0275 102.04)
 		(end 96.0525 102.04)
@@
 	)
 	(segment
+		(start 119.68 56.925)
+		(end 119.725 56.925)
+		(width 0.127)
+		(layer "F.Cu")
+		(net "unconnected-(J1-SHIELD-PadSH)")
+	)
+	(segment
+		(start 119.68 57.32)
+		(end 119.68 61.105)
+		(width 0.127)
+		(layer "F.Cu")
+		(net "unconnected-(J1-SHIELD-PadSH)")
+	)
+	(segment
+		(start 119.9 57.1)
+		(end 119.68 57.32)
+		(width 0.127)
+		(layer "F.Cu")
+		(net "unconnected-(J1-SHIELD-PadSH)")
+	)
+	(segment
+		(start 119.725 56.925)
+		(end 119.9 57.1)
+		(width 0.127)
+		(layer "F.Cu")
+		(net "unconnected-(J1-SHIELD-PadSH)")
+	)
+	(segment
